File: PCB/RP2040 Devboard.kicad_sch (KiCad schematic)
At the start: 37 parts, among them J1 USB_C_Receptacle_USB2.0_16P, J2 Conn_01x02_Pin, J3 Conn_01x04, J4 Conn_01x20, J5 Conn_01x20, SW1 RESET, U1 NCP1117-3.3_TO252, U2 RP2040, U3 W25Q128JVS, Y1 Crystal

Commit message: newer ver. of gerber file
Parts:
- C16, C17: value C -> 27 pF
Changed lines of the file:
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@@
 			)
 		)
-		(property "Value" "C"
+		(property "Value" "27 pF"
 			(at 120.65 140.9699 0)
 			(show_name no)
@@
 			)
 		)
-		(property "Value" "C"
+		(property "Value" "27 pF"
 			(at 114.3 128.2699 0)
 			(show_name no)
